File: weiland-esp32.kicad_pcb (KiCad board)
At the start: 2 copper layers, 68.7 x 21.8 mm, 40 parts, among them CN1 SM05B-SRSS-TB (LF)(SN), CN2 SM04B-SRSS-TB (LF)(SN), CN3 SM04B-SRSS-TB (LF)(SN), CN4 SM02B-SRSS-TB (LF)(SN), CN5 SM02B-SRSS-TB (LF)(SN), U1 ESP32-WROOM-32E(8MB), U2 AMS1117-3.3_C347222, U3 MAX98357AETE_T, U5 ULN2003F12FN-7, U6 DZ127S-22-06-55

Commit message: routed board
Parts:
- moved C9 23.4 mm to (159.1, 30.0), turned to 180 degrees
- moved C5 9.20 mm to (159.1, 25.4), turned to 180 degrees
- moved C4 2.72 mm to (157.5, 33.5), turned to 180 degrees
- moved C1 1.88 mm to (159.1, 27.8), turned to 0 degrees
- moved R2 1.40 mm to (159.1, 28.9), turned to 0 degrees
- moved U2 1.18 mm to (154.2, 28.6)
- moved I14 1.17 mm to (157.8, 42.5)
- moved C2 0.93 mm to (159.1, 26.6), turned to 0 degrees
- moved I15 0.72 mm to (181.1, 43.0)
- moved U3 0.58 mm to (157.9, 37.8)
- moved C6 0.55 mm to (157.5, 35.1)
Routing:
- net GND: track 21.4 -> 9.11 mm, vias 6 -> 2
- net +5V: track 33.1 -> 31.5 mm
- net /EN: track 26.0 -> 27.2 mm
- net /OUTP: track 61.8 -> 60.7 mm, vias 3 -> 2
- net /IO22: track 31.3 -> 32.4 mm
- net /IO14: track 8.29 -> 7.52 mm
- net /IO15: track 26.0 -> 25.4 mm
- net +3.3V: track 51.5 -> 52.0 mm
