File: weiland-esp32.kicad_sch (KiCad schematic)
At the start: 40 parts, among them CN1 SM05B-SRSS-TB (LF)(SN), CN2 SM04B-SRSS-TB (LF)(SN), CN3 SM04B-SRSS-TB (LF)(SN), CN4 SM02B-SRSS-TB (LF)(SN), CN5 SM02B-SRSS-TB (LF)(SN), U1 ESP32-WROOM-32E(8MB), U2 AMS1117-3.3_C347222, U3 MAX98357AETE_T, U5 ULN2003F12FN-7, U6 DZ127S-22-06-55

Commit message: routed board with CC connected to Rd 5.1kohm
Parts:
- added R4: 5.1kOhm, Resistor_SMD:R_0402_1005Metric, symbol 0402WGF5101TCE
- R3: value 56kOhm -> 5.1kOhm
Connections:
- net +5V: no longer R3.2
- net GND: now also R3.2, R4.2
- net at USB1.10 (CC2): now also R4.1
- no-connect marks 28 -> 27
Changed lines of the file:
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@@
 	)
 	(no_connect
-		(at 35.56 63.5)
-	)
-	(no_connect
 		(at 66.04 146.05)
 	)
@@
 	(wire
 		(pts
+			(xy 25.4 63.5) (xy 35.56 63.5)
+		)
+		(stroke
+			(width 0)
+			(type default)
+		)
+	)
+	(wire
+		(pts
 			(xy 93.98 58.42) (xy 100.33 58.42)
 		)
@@
 			)
 		)
-		(property "Value" "56kOhm"
+		(property "Value" "5.1kOhm"
 			(at 22.9997 46.736 0)
 			(effects
@@
 	)
 	(symbol
-		(lib_id "power:+5V")
-		(at 16.51 48.26 90)
+		(lib_id "0402WGF5101TCE")
+		(at 20.32 63.5 90)
 		(unit 1)
 		(exclude_from_sim no)
@@
 		(on_board yes)
 		(dnp no)
-		(fields_autoplaced yes)
-		(property "Reference" "#PWR033"
-			(at 20.32 48.26 0)
+		(property "Reference" "R4"
+			(at 19.4437 61.976 0)
+			(effects
+				(font
+					(face "Arial")
+					(size 1.6891 1.6891)
+				)
+				(justify left top)
+			)
+		)
+		(property "Value" "5.1kOhm"
+			(at 21.7297 61.976 0)
+			(effects
+				(font
+					(face "Arial")
+					(size 1.6891 1.6891)
+				)
+				(justify left top)
+			)
+		)
+		(property "Footprint" "Resistor_SMD:R_0402_1005Metric"
+			(at 20.32 63.5 0)
 			(effects
 				(font
@@
 			)
 		)
-		(property "Value" "+5V"
-			(at 12.7 48.2599 90)
+		(property "Datasheet" ""
+			(at 20.32 63.5 0)
 			(effects
 				(font
 					(size 1.27 1.27)
 				)
-				(justify left)
+				(hide yes)
 			)
 		)
-		(property "Footprint" ""
-			(at 16.51 48.26 0)
+		(property "Description" ""
+			(at 20.32 63.5 0)
 			(effects
 				(font
@@
 			)
 		)
-		(property "Datasheet" ""
-			(at 16.51 48.26 0)
+		(property "Manufacturer Part" "0402WGF5101TCE"
+			(at 20.32 63.5 0)
 			(effects
 				(font
@@
 			)
 		)
-		(property "Description" "Power symbol creates a global label with name \"+5V\""
-			(at 16.51 48.26 0)
+		(property "Manufacturer" "UniOhm"
+			(at 20.32 63.5 0)
+			(effects
+				(font
+					(size 1.27 1.27)
+				)
+				(hide yes)
+			)
+		)
+		(property "Supplier Part" "C25905"
+			(at 20.32 63.5 0)
 			(effects
 				(font
@@
 			)
 		)
+		(property "Supplier" "LCSC"
+			(at 20.32 63.5 0)
+			(effects
+				(font
+					(size 1.27 1.27)
+				)
+				(hide yes)
+			)
+		)
+		(pin "2"
+		)
 		(pin "1"
 		)
@@
 			(project "weiland-esp32"
 				(path "/745a8d65-fa51-45f7-9665-7610e72f2a80"
-					(reference "#PWR033")
+					(reference "R4")
 					(unit 1)
 				)
@@
 	)
 	(symbol
+		(lib_id "power:GND")
+		(at 16.51 48.26 270)
+		(unit 1)
+		(exclude_from_sim no)
+		(in_bom yes)
+		(on_board yes)
+		(dnp no)
+		(fields_autoplaced yes)
+		(property "Reference" "#PWR048"
+			(at 10.16 48.26 0)
+			(effects
+				(font
+					(size 1.27 1.27)
+				)
+				(hide yes)
+			)
+		)
+		(property "Value" "GND"
+			(at 12.7 48.2599 90)
+			(effects
+				(font
+					(size 1.27 1.27)
+				)
+				(justify right)
+			)
+		)
+		(property "Footprint" ""
+			(at 16.51 48.26 0)
+			(effects
+				(font
+					(size 1.27 1.27)
+				)
+				(hide yes)
+			)
+		)
+		(property "Datasheet" ""
+			(at 16.51 48.26 0)
+			(effects
+				(font
+					(size 1.27 1.27)
+				)
+				(hide yes)
+			)
+		)
+		(property "Description" "Power symbol creates a global label with name \"GND\" , ground"
+			(at 16.51 48.26 0)
+			(effects
+				(font
+					(size 1.27 1.27)
+				)
+				(hide yes)
+			)
+		)
+		(pin "1"
+		)
+		(instances
+			(project "weiland-esp32"
+				(path "/745a8d65-fa51-45f7-9665-7610e72f2a80"
+					(reference "#PWR048")
+					(unit 1)
+				)
+			)
+		)
+	)
+	(symbol
 		(lib_id "Connector:TestPoint")
 		(at 368.3 138.43 0)
@@
 					(unit 1)
 				)
+			)
+		)
+	)
+	(symbol
+		(lib_id "power:GND")
+		(at 15.24 63.5 270)
+		(unit 1)
+		(exclude_from_sim no)
+		(in_bom yes)
+		(on_board yes)
+		(dnp no)
+		(fields_autoplaced yes)
+		(property "Reference" "#PWR033"
+			(at 8.89 63.5 0)
+			(effects
+				(font
+					(size 1.27 1.27)
+				)
+				(hide yes)
+			)
+		)
+		(property "Value" "GND"
+			(at 11.43 63.4999 90)
+			(effects
+				(font
+					(size 1.27 1.27)
+				)
+				(justify right)
+			)
+		)
+		(property "Footprint" ""
+			(at 15.24 63.5 0)
+			(effects
+				(font
+					(size 1.27 1.27)
+				)
+				(hide yes)
+			)
+		)
+		(property "Datasheet" ""
+			(at 15.24 63.5 0)
+			(effects
+				(font
+					(size 1.27 1.27)
+				)
+				(hide yes)
+			)
+		)
+		(property "Description" "Power symbol creates a global label with name \"GND\" , ground"
+			(at 15.24 63.5 0)
+			(effects
+				(font
+					(size 1.27 1.27)
+				)
+				(hide yes)
+			)
+		)
+		(pin "1"
+		)
+		(instances
+			(project "weiland-esp32"
+				(path "/745a8d65-fa51-45f7-9665-7610e72f2a80"
+					(reference "#PWR033")
+					(unit 1)
+				)

Commit message: capacitors for ULN2003 and co and coin motors
Parts:
- added C10: 1uF, Capacitor_SMD:C_0402_1005Metric, symbol Device:C
- added C11, C12, C13, C14: 100nF, Capacitor_SMD:C_0402_1005Metric, symbol Device:C_Small
Connections:
- net +5V: now also U5.6 (COM), C10.2, C11.1, C12.1, C13.1, C14.1
- net GND: now also C10.1
- net OUTA: now also C13.2
- net OUTB: now also C14.2
- net OUTC: now also C12.2
- net OUTD: now also C11.2
- no-connect marks 27 -> 26
